Commit message: Tilted realsense camera

File: yahboom_rosmaster_description/urdf/robots/rosmaster_x3.urdf.xacro (robot description, xacro)
@@ -29,5 +29,5 @@
       prefix="$(arg prefix)"
       camera_name="cam_1"
-      xyz_offset="0.0 0 0.1"
-      rpy_offset="0 0.2 0"/>
+      xyz_offset="0.09 0 0.05"
+      rpy_offset="0 -0.55 0"/>
 </robot>

File: yahboom_rosmaster_description/urdf/sensors/rgbd_camera.urdf.xacro (robot description, xacro)
@@ -7,6 +7,6 @@
     parent:='base_link'
     mesh_file:='file://$(find yahboom_rosmaster_description)/meshes/intel_realsense/visual/d435.stl'
-    xyz_offset:='0 0.01 0.50'
-    rpy_offset:='0.0 ${45 * M_PI/180} ${M_PI/2}'
+    xyz_offset:='0.09 0 0.05'
+    rpy_offset:='0 -0.55 0'
     mesh_xyz_offset:='0 0 0'
     mesh_rpy_offset:='${M_PI/2} 0.0 ${M_PI/2}'
@@ -44,5 +44,6 @@
     update_rate:=5
     always_on:=1
-    visualize:=true">
+    visualize:=true
+    enable_collision:=false">
     <link name="${prefix}${camera_name}_link">
       <visual>
@@ -55,10 +56,12 @@
         </material>
       </visual>
-      <collision>
-        <origin xyz="${collision_xyz_offset}" rpy="${collision_rpy_offset}"/>
-        <geometry>
-          <box size="${cam_depth} ${cam_width} ${cam_height}"/>
-        </geometry>
-      </collision>
+      <xacro:if value="${enable_collision}">
+        <collision>
+          <origin xyz="${collision_xyz_offset}" rpy="${collision_rpy_offset}"/>
+          <geometry>
+            <box size="${cam_depth} ${cam_width} ${cam_height}"/>
+          </geometry>
+        </collision>
+      </xacro:if>
       <inertial>
         <mass value="${mass}" />

Commit message: Added LIDAR to URDF

File: yahboom_rosmaster_description/urdf/robots/rosmaster_x3.urdf.xacro (robot description, xacro)
@@ -1,8 +1,10 @@
 <?xml version="1.0"?>
 <robot xmlns:xacro="http://www.ros.org/wiki/xacro" name="rosmaster_x3">
+    <xacro:property name="M_PI" value="3.1415926535897931" />
     <xacro:arg name="prefix" default=""/>
     <xacro:include filename="$(find yahboom_rosmaster_description)/urdf/mech/rosmaster_x3_base.urdf.xacro"/>
     <xacro:include filename="$(find yahboom_rosmaster_description)/urdf/mech/mecanum_wheel.urdf.xacro"/>
     <xacro:include filename="$(find yahboom_rosmaster_description)/urdf/sensors/rgbd_camera.urdf.xacro"/>
+    <xacro:include filename="$(find yahboom_rosmaster_description)/urdf/sensors/lidar.urdf.xacro"/>
     <xacro:rosmaster_x3_base prefix="$(arg prefix)"/>
     <xacro:mecanum_wheel
@@ -29,5 +31,13 @@
       prefix="$(arg prefix)"
       camera_name="cam_1"
-      xyz_offset="0.09 0 0.05"
-      rpy_offset="0 -0.55 0"/>
+      xyz_offset="0.105 0 0.05"
+      rpy_offset="0 -0.50 0"/>
+    <xacro:lidar_sensor
+      prefix="$(arg prefix)"
+      parent="base_link"
+      frame_id="laser_frame"
+      xyz_offset="0 0 0.0825"
+      rpy_offset="0 0 0"
+      mesh_xyz_offset="0 0 0"
+      mesh_rpy_offset="${-M_PI/2} 0 0"/>
 </robot>

File: yahboom_rosmaster_description/urdf/sensors/rgbd_camera.urdf.xacro (robot description, xacro)
@@ -7,6 +7,6 @@
     parent:='base_link'
     mesh_file:='file://$(find yahboom_rosmaster_description)/meshes/intel_realsense/visual/d435.stl'
-    xyz_offset:='0.09 0 0.05'
-    rpy_offset:='0 -0.55 0'
+    xyz_offset:='0.105 0 0.05'
+    rpy_offset:='0 -0.50 0'
     mesh_xyz_offset:='0 0 0'
     mesh_rpy_offset:='${M_PI/2} 0.0 ${M_PI/2}'

Commit message: Add IMU to main URDF

File: yahboom_rosmaster_description/urdf/robots/rosmaster_x3.urdf.xacro (robot description, xacro)
@@ -7,4 +7,5 @@
     <xacro:include filename="$(find yahboom_rosmaster_description)/urdf/sensors/rgbd_camera.urdf.xacro"/>
     <xacro:include filename="$(find yahboom_rosmaster_description)/urdf/sensors/lidar.urdf.xacro"/>
+    <xacro:include filename="$(find yahboom_rosmaster_description)/urdf/sensors/imu.urdf.xacro"/>
     <xacro:rosmaster_x3_base prefix="$(arg prefix)"/>
     <xacro:mecanum_wheel
@@ -40,4 +41,13 @@
       rpy_offset="0 0 0"
       mesh_xyz_offset="0 0 0"
-      mesh_rpy_offset="${-M_PI/2} 0 0"/>
+      mesh_rpy_offset="${-M_PI/2} 0 0"
+      topic_name="scan"/>
+    <xacro:imu_sensor
+      prefix="$(arg prefix)"
+      parent="base_link"
+      frame_id="imu"
+      xyz_offset="0 0 0.006"
+      rpy_offset="0 0 0"
+      update_rate="15.0"
+      topic_name="imu/data"/>
 </robot>

File: yahboom_rosmaster_description/urdf/sensors/imu.urdf.xacro (robot description, xacro)
@@ -10,8 +10,8 @@
         inertial_xyz_offset:='0 0 0'
         inertial_rpy_offset:='0 0 0'
-        mass:='0.031'
-        length:='0.03899'
-        width:='0.03785'
-        height:='0.01338'
+        mass:=0.031
+        length:=0.03899
+        width:=0.03785
+        height:=0.01338
         material_name:='imu_black'
         material_color:='0.1 0.1 0.1 1'
@@ -23,7 +23,7 @@
         always_on:=true
         visualize:=false">
-        <xacro:property name="ixx" value="${(mass/12) * (height*height + width*width)}" />
-        <xacro:property name="iyy" value="${(mass/12) * (length*length + height*height)}" />
-        <xacro:property name="izz" value="${(mass/12) * (length*length + width*width)}" />
+        <xacro:property name="ixx" value="${(mass/12.0) * (height*height + width*width)}" />
+        <xacro:property name="iyy" value="${(mass/12.0) * (length*length + height*height)}" />
+        <xacro:property name="izz" value="${(mass/12.0) * (length*length + width*width)}" />
         <link name="${prefix}${frame_id}_link">
             <visual>
