Commit message: Removed comments from URDF

File: yahboom_rosmaster_description/urdf/mech/rosmaster_x3_base.urdf.xacro (robot description, xacro)
@@ -5,7 +5,7 @@
 <xacro:property name="wheel_radius" value="0.0325" />
 <xacro:property name="total_height" value="0.26225" />
-<xacro:property name="base_length" value="0.300" />  <!-- 300mm -->
-<xacro:property name="centered_length" value="0.238" />  <!-- 238mm -->
-<xacro:property name="base_x_offset" value="${(centered_length - base_length) / 2}" />  <!-- (238-300)/2 mm in meters -->
+<xacro:property name="base_length" value="0.300" />
+<xacro:property name="centered_length" value="0.238" />
+<xacro:property name="base_x_offset" value="${(centered_length - base_length) / 2}" />
 <xacro:property name="base_size_x" value="${base_length}" />
 <xacro:property name="base_size_y" value="${total_width - (2 * wheel_width)}" />

Commit message: Make the base green

File: yahboom_rosmaster_description/urdf/mech/rosmaster_x3_base.urdf.xacro (robot description, xacro)
@@ -19,4 +19,7 @@
             <mesh filename="file://$(find yahboom_rosmaster_description)/meshes/rosmaster_x3/visual/base_link_X3.STL"/>
         </geometry>
+        <material name="green">
+          <color rgba="0 0.7 0 1"/>
+        </material>
         <origin xyz="0 0 0" rpy="0 0 0"/>
     </visual>

Commit message: Add mecanum wheels

File: yahboom_rosmaster_description/urdf/mech/rosmaster_x3_base.urdf.xacro (robot description, xacro)
@@ -28,8 +28,8 @@
             <box size="${base_size_x} ${base_size_y} ${base_size_z}"/>
         </geometry>
-        <origin xyz="${base_x_offset} 0 ${base_size_z/2}" rpy="0 0 0"/>
+        <origin xyz="${base_x_offset} 0 ${base_size_z/2 + wheel_radius/4}" rpy="0 0 0"/>
     </collision>
     <inertial>
-        <origin xyz="${base_x_offset} 0 ${base_size_z/2}" rpy="0 0 0"/>
+        <origin xyz="${base_x_offset} 0 ${base_size_z/2 + wheel_radius/4}" rpy="0 0 0"/>
         <mass value="${base_mass}"/>
         <inertia

File: yahboom_rosmaster_description/urdf/robots/rosmaster_x3.urdf.xacro (robot description, xacro)
@@ -3,4 +3,25 @@
     <xacro:arg name="prefix" default=""/>
     <xacro:include filename="$(find yahboom_rosmaster_description)/urdf/mech/rosmaster_x3_base.urdf.xacro"/>
+    <xacro:include filename="$(find yahboom_rosmaster_description)/urdf/mech/mecanum_wheel.urdf.xacro"/>
     <xacro:rosmaster_x3_base prefix="$(arg prefix)"/>
+    <xacro:mecanum_wheel
+        prefix="$(arg prefix)"
+        side="front_right"
+        x_reflect="-1"
+        y_reflect="1"/>
+    <xacro:mecanum_wheel
+        prefix="$(arg prefix)"
+        side="front_left"
+        x_reflect="-1"
+        y_reflect="-1"/>
+    <xacro:mecanum_wheel
+        prefix="$(arg prefix)"
+        side="back_left"
+        x_reflect="1"
+        y_reflect="-1"/>
+    <xacro:mecanum_wheel
+        prefix="$(arg prefix)"
+        side="back_right"
+        x_reflect="1"
+        y_reflect="1"/>
 </robot>

Commit message: Removed base footprint from URDF

File: yahboom_rosmaster_description/urdf/mech/rosmaster_x3_base.urdf.xacro (robot description, xacro)
@@ -13,5 +13,4 @@
 <xacro:property name="base_mass" value="4.6" />
 <xacro:macro name="rosmaster_x3_base" params="prefix">
-  <link name="${prefix}base_footprint"/>
   <link name="${prefix}base_link">
     <visual>
@@ -48,9 +47,4 @@
     </visual>
   </gazebo>
-  <joint name="${prefix}base_joint" type="fixed">
-    <parent link="${prefix}base_footprint"/>
-    <child link="${prefix}base_link"/>
-    <origin xyz="0 0 ${wheel_radius}" rpy="0 0 0"/>
-  </joint>
 </xacro:macro>
 </robot>

Commit message: Updated to add back base footprint

File: yahboom_rosmaster_description/urdf/mech/rosmaster_x3_base.urdf.xacro (robot description, xacro)
@@ -13,4 +13,5 @@
 <xacro:property name="base_mass" value="4.6" />
 <xacro:macro name="rosmaster_x3_base" params="prefix">
+  <link name="${prefix}base_footprint"/>
   <link name="${prefix}base_link">
     <visual>
@@ -47,4 +48,9 @@
     </visual>
   </gazebo>
+  <joint name="${prefix}base_joint" type="fixed">
+    <parent link="${prefix}base_footprint"/>
+    <child link="${prefix}base_link"/>
+    <origin xyz="0 0 ${wheel_radius}" rpy="0 0 0"/>
+  </joint>
 </xacro:macro>
 </robot>
