Commit message: Make torsional friction 0 in wheel URDF

File: yahboom_rosmaster_description/urdf/mech/mecanum_wheel.urdf.xacro (robot description, xacro)
@@ -40,17 +40,37 @@
     </joint>
     <gazebo reference="${prefix}${side}_wheel_link">
-      <mu1>0.01</mu1>
-      <mu2>0.01</mu2>
+      <surface>
+          <friction>
+              <ode>
+                  <mu>0.01</mu>
+                  <mu2>0.01</mu2>
+              </ode>
+              <torsional>
+                  <coefficient>0.0</coefficient>
+              </torsional>
+          </friction>
+      </surface>
     </gazebo>
     <gazebo reference="${prefix}${side}_wheel_link">
+      <surface>
+          <friction>
+              <ode>
+                  <mu>0.01</mu>
+                  <mu2>0.01</mu2>
+              </ode>
+              <torsional>
+                  <coefficient>0.0</coefficient>
+              </torsional>
+          </friction>
+      </surface>
       <visual>
-        <material>
-          <ambient>0.2 0.2 0.2 1.0</ambient>
-          <diffuse>0.2 0.2 0.2 1.0</diffuse>
-          <specular>0.2 0.2 0.2 1.0</specular>
-          <emissive>0.0 0.0 0.0 0.0</emissive>
-        </material>
+          <material>
+              <ambient>0.2 0.2 0.2 1.0</ambient>
+              <diffuse>0.2 0.2 0.2 1.0</diffuse>
+              <specular>0.2 0.2 0.2 1.0</specular>
+              <emissive>0.0 0.0 0.0 0.0</emissive>
+          </material>
       </visual>
-    </gazebo>
+  </gazebo>
   </xacro:macro>
 </robot>

Commit message: Added unrealistic mass to wheels to make robot behave better in Gazebo

File: yahboom_rosmaster_description/urdf/mech/mecanum_wheel.urdf.xacro (robot description, xacro)
@@ -4,5 +4,5 @@
   <xacro:property name="wheel_separation" value="0.169" />
   <xacro:property name="wheel_width" value="0.03040" />
-  <xacro:property name="wheel_mass" value="0.1" />
+  <xacro:property name="wheel_mass" value="9.1" />
   <xacro:property name="wheel_xoff" value="0.08" />
   <xacro:property name="wheel_yoff" value="-0.01" />
